File: hardware/Eagle PCB/AnalogKeyPad.brd (EAGLE design)
At the start: 40 x 50 mm, 13 parts

Commit message: update hardware
Parts:
- removed C2: 10uF, rcl2:E2,5-6E
Connections:
- net GND: now also C1.1; no longer C2.-, SV1.3
- net VCC: no longer C1.1, C2.+
Routing:
- net VCC: track 26.0 -> 17.7 mm
- net A0: track 70.9 -> 68.6 mm
Changed lines of the file:
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@@
 <attribute name="MF" value="" x="20" y="47.5" size="1.778" layer="27" display="off"/>
 </element>
-<element name="C2" library="rcl2" package="E2,5-6E" value="10uF" x="4" y="45" rot="R180"/>
 </elements>
 <signals>
-<signal name="VCC">
-<contactref element="C1" pad="1"/>
-<contactref element="R1" pad="2"/>
-<contactref element="SV1" pad="1"/>
-<wire x1="4" y1="41.81" x2="4" y2="43" width="0.8128" layer="16"/>
-<wire x1="4" y1="43" x2="6.615384375" y2="46.923078125" width="0.8128" layer="16"/>
-<wire x1="6.615384375" y1="46.923078125" x2="7" y2="47.5" width="0.8128" layer="16"/>
-<wire x1="7" y1="47.5" x2="17.46" y2="47.5" width="0.8128" layer="16"/>
-<wire x1="7.62" y1="39.37" x2="4.63" y2="39.37" width="0.8128" layer="16"/>
-<wire x1="4.63" y1="39.37" x2="4" y2="40" width="0.8128" layer="16"/>
-<wire x1="4" y1="40" x2="4" y2="41.81" width="0.8128" layer="16"/>
-<contactref element="C2" pad="+"/>
-<wire x1="5.27" y1="45" x2="6.5" y2="45" width="0.8128" layer="16"/>
-<wire x1="6.5" y1="45" x2="6.5" y2="46" width="0.8128" layer="16"/>
-<wire x1="6.5" y1="46" x2="6.615384375" y2="46" width="0.8128" layer="16"/>
-<wire x1="6.615384375" y1="46" x2="6.615384375" y2="46.923078125" width="0.8128" layer="16"/>
-</signal>
 <signal name="A0">
 <contactref element="R1" pad="1"/>
 <contactref element="R2" pad="2"/>
-<contactref element="C1" pad="2"/>
 <contactref element="DOWN" pad="1"/>
-<contactref element="SV1" pad="2"/>
 <wire x1="4" y1="34.19" x2="7.52" y2="34.19" width="0.8128" layer="16"/>
-<wire x1="7.52" y1="34.19" x2="7.62" y2="34.29" width="0.8128" layer="16"/>
 <wire x1="6" y1="8" x2="4" y2="10" width="0.8128" layer="16"/>
 <wire x1="4" y1="10" x2="4" y2="34.19" width="0.8128" layer="16"/>
-<wire x1="7.62" y1="34.29" x2="7.79" y2="34.29" width="0.8128" layer="16"/>
 <wire x1="7.79" y1="34.29" x2="9.5" y2="36" width="0.8128" layer="16"/>
 <wire x1="9.5" y1="36" x2="9.5" y2="37.5" width="0.8128" layer="16"/>
@@
 <wire x1="13" y1="44.5" x2="19" y2="44.5" width="0.8128" layer="16"/>
 <wire x1="19" y1="44.5" x2="20" y2="45.5" width="0.8128" layer="16"/>
-<wire x1="20" y1="45.5" x2="20" y2="47.5" width="0.8128" layer="16"/>
 <contactref element="DOWN" pad="2"/>
 <wire x1="17.7394" y1="9.2512" x2="17.7394" y2="8" width="0.8128" layer="16"/>
 <wire x1="17.7394" y1="8" x2="17.7394" y2="2.7488" width="0.8128" layer="16"/>
 <wire x1="6" y1="8" x2="17.7394" y2="8" width="0.8128" layer="16"/>
+<contactref element="SV1" pad="2"/>
+<contactref element="C1" pad="2"/>
+<wire x1="20" y1="45.5" x2="20" y2="47.5" width="0" layer="19" extent="16-16"/>
+<wire x1="7.62" y1="34.29" x2="7.79" y2="34.29" width="0" layer="19" extent="16-16"/>
+<wire x1="7.52" y1="34.19" x2="7.62" y2="34.29" width="0" layer="19" extent="16-16"/>
 </signal>
 <signal name="N$2">
@@
 <contactref element="LEFT" pad="3"/>
 <contactref element="RIGHT" pad="3"/>
-<contactref element="SV1" pad="3"/>
 <polygon width="0.4064" layer="16">
 <vertex x="0" y="50"/>
@@
 <contactref element="LEFT" pad="4"/>
 <contactref element="DOWN" pad="4"/>
-<contactref element="C2" pad="-"/>
+<contactref element="C1" pad="1"/>
 </signal>
 <signal name="N$4">
@@
 <wire x1="32.2606" y1="19.2512" x2="32.2606" y2="12.7488" width="0.8128" layer="16"/>
 </signal>
+<signal name="VCC">
+<contactref element="SV1" pad="1"/>
+<contactref element="R1" pad="2"/>
+<wire x1="17.46" y1="47.5" x2="6.5" y2="47.5" width="0.8128" layer="16"/>
+<wire x1="6.5" y1="47.5" x2="4" y2="45" width="0.8128" layer="16"/>
+<wire x1="4" y1="45" x2="4" y2="41.81" width="0.8128" layer="16"/>
+</signal>
 </signals>
