File: hardware/Eagle PCB/AnalogKeyPad.sch (EAGLE design)
At the start: 13 parts

Commit message: update hardware
Parts:
- removed C2: 10uF, rcl2:CPOL-USE2,5-6E
Connections:
- net GND: now also C1.1; no longer C2.-, SV1.3
- net VCC: no longer C1.1, C2.+
Other:
- moved on the sheet: C1, SV1
Changed lines of the file:
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@@
 <part name="LEFT" library="switch-omron" deviceset="10-XX" device=""/>
 <part name="SV1" library="con-lstb" deviceset="MA03-1" device=""/>
-<part name="C2" library="rcl2" deviceset="CPOL-US" device="E2,5-6E" value="10uF"/>
-<part name="P+2" library="supply1" deviceset="VCC" device=""/>
 <part name="GND2" library="supply1" deviceset="GND" device=""/>
 </parts>
@@
 <instance part="R4" gate="G$1" x="78.74" y="35.56" rot="R90"/>
 <instance part="R5" gate="G$1" x="78.74" y="20.32" rot="R90"/>
-<instance part="C1" gate="G$1" x="93.98" y="86.36"/>
-<instance part="P+1" gate="VCC" x="93.98" y="96.52"/>
-<instance part="GND1" gate="1" x="50.8" y="-2.54"/>
+<instance part="C1" gate="G$1" x="88.9" y="68.58" rot="R180"/>
+<instance part="P+1" gate="VCC" x="78.74" y="93.98"/>
+<instance part="GND1" gate="1" x="50.8" y="2.54"/>
 <instance part="DOWN" gate="1" x="60.96" y="76.2" rot="R270"/>
 <instance part="RIGHT" gate="1" x="60.96" y="60.96" rot="R270"/>
@@
 <instance part="UP" gate="1" x="60.96" y="27.94" rot="R270"/>
 <instance part="LEFT" gate="1" x="60.96" y="10.16" rot="R270"/>
-<instance part="SV1" gate="G$1" x="124.46" y="68.58" rot="R180"/>
-<instance part="C2" gate="G$1" x="99.06" y="45.72"/>
-<instance part="P+2" gate="VCC" x="99.06" y="55.88"/>
-<instance part="GND2" gate="1" x="99.06" y="33.02"/>
+<instance part="SV1" gate="G$1" x="109.22" y="76.2" rot="R180"/>
+<instance part="GND2" gate="1" x="88.9" y="60.96"/>
 </instances>
 <busses>
 </busses>
 <nets>
-<net name="VCC" class="0">
-<segment>
-<pinref part="P+1" gate="VCC" pin="VCC"/>
-<pinref part="C1" gate="G$1" pin="1"/>
-<wire x1="93.98" y1="93.98" x2="93.98" y2="91.44" width="0.1524" layer="91"/>
-<pinref part="R1" gate="G$1" pin="2"/>
-<wire x1="93.98" y1="91.44" x2="93.98" y2="88.9" width="0.1524" layer="91"/>
-<wire x1="78.74" y1="88.9" x2="78.74" y2="91.44" width="0.1524" layer="91"/>
-<wire x1="78.74" y1="91.44" x2="93.98" y2="91.44" width="0.1524" layer="91"/>
-</segment>
-<segment>
-<pinref part="SV1" gate="G$1" pin="1"/>
-<wire x1="114.3" y1="71.12" x2="116.84" y2="71.12" width="0.1524" layer="91"/>
-<label x="114.3" y="71.12" size="1.016" layer="95" rot="R180" xref="yes"/>
-</segment>
-<segment>
-<pinref part="C2" gate="G$1" pin="+"/>
-<pinref part="P+2" gate="VCC" pin="VCC"/>
-<wire x1="99.06" y1="53.34" x2="99.06" y2="48.26" width="0.1524" layer="91"/>
-</segment>
-</net>
 <net name="A0" class="0">
 <segment>
@@
 <pinref part="R2" gate="G$1" pin="2"/>
 <wire x1="78.74" y1="78.74" x2="78.74" y2="76.2" width="0.1524" layer="91"/>
-<pinref part="C1" gate="G$1" pin="2"/>
 <wire x1="78.74" y1="76.2" x2="78.74" y2="73.66" width="0.1524" layer="91"/>
-<wire x1="93.98" y1="81.28" x2="93.98" y2="76.2" width="0.1524" layer="91"/>
-<wire x1="93.98" y1="76.2" x2="78.74" y2="76.2" width="0.1524" layer="91"/>
+<wire x1="101.6" y1="76.2" x2="88.9" y2="76.2" width="0.1524" layer="91"/>
 <junction x="78.74" y="76.2"/>
 <pinref part="DOWN" gate="1" pin="S"/>
+<wire x1="88.9" y1="76.2" x2="78.74" y2="76.2" width="0.1524" layer="91"/>
 <wire x1="66.04" y1="76.2" x2="78.74" y2="76.2" width="0.1524" layer="91"/>
-<wire x1="93.98" y1="76.2" x2="99.06" y2="76.2" width="0.1524" layer="91"/>
-<junction x="93.98" y="76.2"/>
-<label x="99.06" y="76.2" size="1.016" layer="95" xref="yes"/>
 <pinref part="DOWN" gate="1" pin="S1"/>
 <wire x1="66.04" y1="73.66" x2="66.04" y2="76.2" width="0.1524" layer="91"/>
-</segment>
-<segment>
 <pinref part="SV1" gate="G$1" pin="2"/>
-<wire x1="116.84" y1="68.58" x2="114.3" y2="68.58" width="0.1524" layer="91"/>
-<label x="114.3" y="68.58" size="1.016" layer="95" rot="R180" xref="yes"/>
+<pinref part="C1" gate="G$1" pin="2"/>
+<wire x1="88.9" y1="73.66" x2="88.9" y2="76.2" width="0.1524" layer="91"/>
+<junction x="88.9" y="76.2"/>
 </segment>
 </net>
@@
 <wire x1="50.8" y1="43.18" x2="50.8" y2="27.94" width="0.1524" layer="91"/>
 <wire x1="50.8" y1="27.94" x2="50.8" y2="10.16" width="0.1524" layer="91"/>
-<wire x1="50.8" y1="10.16" x2="50.8" y2="0" width="0.1524" layer="91"/>
+<wire x1="50.8" y1="10.16" x2="50.8" y2="5.08" width="0.1524" layer="91"/>
 <wire x1="55.88" y1="43.18" x2="50.8" y2="43.18" width="0.1524" layer="91"/>
 <pinref part="UP" gate="1" pin="P"/>
@@
 </segment>
 <segment>
-<pinref part="SV1" gate="G$1" pin="3"/>
-<wire x1="116.84" y1="66.04" x2="114.3" y2="66.04" width="0.1524" layer="91"/>
-<label x="114.3" y="66.04" size="1.016" layer="95" rot="R180" xref="yes"/>
-</segment>
-<segment>
-<pinref part="C2" gate="G$1" pin="-"/>
+<pinref part="C1" gate="G$1" pin="1"/>
 <pinref part="GND2" gate="1" pin="GND"/>
-<wire x1="99.06" y1="40.64" x2="99.06" y2="35.56" width="0.1524" layer="91"/>
+<wire x1="88.9" y1="66.04" x2="88.9" y2="63.5" width="0.1524" layer="91"/>
 </segment>
 </net>
@@
 </segment>
 </net>
+<net name="VCC" class="0">
+<segment>
+<pinref part="SV1" gate="G$1" pin="1"/>
+<wire x1="101.6" y1="78.74" x2="88.9" y2="78.74" width="0.1524" layer="91"/>
+<wire x1="88.9" y1="78.74" x2="88.9" y2="91.44" width="0.1524" layer="91"/>
+<pinref part="P+1" gate="VCC" pin="VCC"/>
+<wire x1="88.9" y1="91.44" x2="78.74" y2="91.44" width="0.1524" layer="91"/>
+<pinref part="R1" gate="G$1" pin="2"/>
+<wire x1="78.74" y1="91.44" x2="78.74" y2="88.9" width="0.1524" layer="91"/>
+<junction x="78.74" y="91.44"/>
+</segment>
+</net>
