File: hardware/KiCAD PCB/lader keypad.kicad_pcb (KiCad board)
At the start: 2 copper layers, 50 x 50 mm, 13 parts, among them J1 CONNECTOR, SW1 Down, SW2 Left, SW3 Select, SW4 Up, SW5 Right

Commit message: update hardware
Parts:
- removed C2: 10uF/16v, Capacitors_ThroughHole:CP_Radial_D6.3mm_P2.50mm
Connections:
- C1 pad 1: +5V -> GND
Routing:
- net +5V: track 47.1 -> 16.0 mm
